Commit message: Disabled finger spread joints

File: genesis/assets/urdf/wam_description/urdf/wam.urdf (robot description, URDF)
Before this commit: robot wam, 20 links, 19 joints
Joints:
- joint bhand_spread: axis 0 0 -1 -> (none); limit lower=0.0 upper=3.14159265359 effort=30 velocity=2.0 -> (none); type revolute -> fixed
- joint bhand_spread_finger2: axis 0 0 1 -> (none); limit lower=0.0 upper=3.14159265359 effort=30 velocity=2.0 -> (none); mimic joint=bhand_spread multiplier=1.0 offset=0 -> (none); type revolute -> fixed
