Commit message: Changed fingers to boxes and adjusted wrist angle

File: wam/wam_description/urdf/wam_finger.urdf (robot description, URDF)
Before this commit: robot wam, 20 links, 19 joints
Links:
- link bhand_finger1_link_1: geometry collision box size=0.1 0.02 0.02; visual box size=0.1 0.02 0.02
- link bhand_finger1_link_2: geometry collision box size=0.1 0.02 0.02; visual box size=0.1 0.02 0.02
- link bhand_finger1_link_3: geometry collision box size=0.1 0.02 0.02; visual box size=0.1 0.02 0.02
- link bhand_finger2_link_1: geometry collision box size=0.1 0.02 0.02; visual box size=0.1 0.02 0.02
- link bhand_finger2_link_2: geometry collision box size=0.1 0.02 0.02; visual box size=0.1 0.02 0.02
- link bhand_finger2_link_3: geometry collision box size=0.1 0.02 0.02; visual box size=0.1 0.02 0.02
- link bhand_finger3_link_1: geometry collision box size=0.1 0.02 0.02; visual box size=0.1 0.02 0.02
- link bhand_finger3_link_2: geometry collision box size=0.1 0.02 0.02; visual box size=0.1 0.02 0.02
- link bhand_finger3_link_3: geometry collision box size=0.1 0.02 0.02; visual box size=0.1 0.02 0.02
Joints:
- joint wam_joint_7: limit lower=-3.0 upper=3.0 effort=30 velocity=2.0 -> lower=-1.5 upper=1.5 effort=30 velocity=2.0

Commit message: modified finger collison

File: wam/wam_description/urdf/wam_finger.urdf (robot description, URDF)
Before this commit: robot wam, 20 links, 19 joints
Links:
- link bhand_finger1_link_1: geometry collision box size=0.08 0.025 0.05; visual mesh filename=package://wam_description/mesh/bh_link1.stl scale=1.0 1.0 1.0
- link bhand_finger1_link_2: geometry collision box size=0.092 0.027 0.02; visual mesh filename=package://wam_description/mesh/bh_link2.stl scale=1.0 1.0 1.0
- link bhand_finger1_link_3: geometry collision box size=0.066 0.019 0.023; visual mesh filename=package://wam_description/mesh/bh_link3.stl scale=1.0 1.0 1.0
- link bhand_finger2_link_1: geometry collision box size=0.08 0.025 0.05; visual mesh filename=package://wam_description/mesh/bh_link1.stl scale=1.0 1.0 1.0
- link bhand_finger2_link_2: geometry collision box size=0.092 0.027 0.02; visual mesh filename=package://wam_description/mesh/bh_link2.stl scale=1.0 1.0 1.0
- link bhand_finger2_link_3: geometry collision box size=0.066 0.019 0.023; visual mesh filename=package://wam_description/mesh/bh_link3.stl scale=1.0 1.0 1.0
- link bhand_finger3_link_1: geometry collision box size=0.08 0.025 0.05; visual mesh filename=package://wam_description/mesh/bh_link1.stl scale=1.0 1.0 1.0
- link bhand_finger3_link_2: geometry collision box size=0.092 0.027 0.02; visual mesh filename=package://wam_description/mesh/bh_link2.stl scale=1.0 1.0 1.0
- link bhand_finger3_link_3: geometry collision box size=0.066 0.019 0.023; visual mesh filename=package://wam_description/mesh/bh_link3.stl scale=1.0 1.0 1.0
